File: hardware/controller.brd (EAGLE design)
At the start: 94.1 x 81.3 mm, 5 parts

Commit message: i
Routing:
- net N$1: track 94.1 -> 0.00 mm
Changed lines of the file:
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@@
 <text x="91.44" y="72.39" size="1.4224" layer="21" rot="R180">github.com/matthewvilim/featherctrl</text>
 <text x="91.44" y="74.93" size="1.4224" layer="21" rot="R180">Matthew Vilim</text>
+<wire x1="0" y1="0" x2="94.06" y2="0" width="0" layer="20"/>
 </plain>
 <attributes>
@@
 <wire x1="5" y1="76.12" x2="5" y2="32.89" width="0.2032" layer="1"/>
 <wire x1="55.88" y1="77.47" x2="53.34" y2="80.01" width="0.2032" layer="1"/>
-<wire x1="8.89" y1="80.01" x2="5" y2="76.12" width="0.2032" layer="1"/>
+<wire x1="5" y1="76.12" x2="8.89" y2="80.01" width="0.2032" layer="1"/>
 </signal>
 <signal name="COL_L">
@@
 <contactref element="U$1" pad="2"/>
 </signal>
-<signal name="N$1">
-<wire x1="0" y1="0" x2="94.06" y2="0" width="0" layer="16"/>
-</signal>
 <signal name="3V2">

Commit message: i
Parts:
- U$1: device mike:NRF52FEATHER -> adafruit:NRF52FEATHER
- flipped U$4 to the top, turned to 0 degrees
- flipped U$7 to the top
Connections:
- removed net N$19: U$5.P$9
- removed net N$24: U$5.P$4
- removed net N$44: U$4.P$5
- removed net N$50: U$4.P$11
- removed net N$54: U$6.P$13
- removed net N$55: U$6.P$11
- removed net N$56: U$6.P$12
- removed net N$57: U$6.P$10
- removed net N$58: U$6.P$9
- removed net N$60: U$6.P$7
- removed net N$61: U$6.P$6
- removed net N$67: U$7.P$1
- removed net N$68: U$7.P$2
- removed net N$75: U$7.P$9
- removed net N$76: U$7.P$10
- removed net N$77: U$7.P$11
- removed net N$78: U$7.P$12
- removed net N$79: U$7.P$13
- net COL_G: now also U$4.P$13, U$7.P$11; no longer U$4.P$1, U$7.P$3
- net COL_H: now also U$4.P$11, U$7.P$10; no longer U$4.P$3, U$7.P$4
- net COL_I: now also U$4.P$12, U$7.P$9; no longer U$4.P$2, U$7.P$5
- net COL_J: now also U$4.P$2, U$7.P$8; no longer U$4.P$12, U$7.P$6
- net COL_K: now also U$4.P$1; no longer U$4.P$13
- net COL_L: now also U$4.P$8; no longer U$4.P$6
- net ROW_1: now also U$4.P$4; no longer U$4.P$10
- net ROW_2: now also U$4.P$5; no longer U$4.P$9
- net ROW_3: now also U$4.P$6; no longer U$4.P$8
- net ROW_5: now also U$4.P$10; no longer U$4.P$4
- net ROW_6: now also U$7.P$6; no longer U$7.P$8
