File: hardware/controller.brd (EAGLE design)
At the start: 94.1 x 81.3 mm, 5 parts

Commit message: i
Connections:
- net 3V renamed 3V1
Routing:
- net COL_K: track 106.9 -> 101.0 mm
- net COL_J: track 140.7 -> 135.5 mm
- net ROW_1: track 98.3 -> 93.9 mm
- net ROW_2: track 176.2 -> 172.5 mm
- net ROW_3: track 174.8 -> 171.8 mm
- net ROW_4: track 179.5 -> 177.2 mm
- net ROW_5: track 174.1 -> 172.6 mm
- net COL_L: track 82.9 -> 81.4 mm
- net COL_H: track 95.6 -> 94.8 mm
Changed lines of the file:
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@@
 <contactref element="U$1" pad="7"/>
 <wire x1="8.89" y1="74.93" x2="11.43" y2="77.47" width="0.2032" layer="1"/>
-<wire x1="48.26" y1="77.47" x2="50.8" y2="74.93" width="0.2032" layer="1"/>
-<wire x1="50.8" y1="74.93" x2="50.8" y2="67.31" width="0.2032" layer="1"/>
 <wire x1="8.89" y1="31.38" x2="8.89" y2="74.93" width="0.2032" layer="1"/>
-<wire x1="11.43" y1="77.47" x2="48.26" y2="77.47" width="0.2032" layer="1"/>
 <contactref element="U$4" pad="P$4"/>
 <wire x1="6.65" y1="29.16" x2="8.87" y2="31.38" width="0.2032" layer="1"/>
 <wire x1="8.87" y1="31.38" x2="8.89" y2="31.38" width="0.2032" layer="1"/>
+<wire x1="11.43" y1="77.47" x2="40.64" y2="77.47" width="0.2032" layer="1"/>
+<wire x1="40.64" y1="77.47" x2="50.8" y2="67.31" width="0.2032" layer="1"/>
 </signal>
 <signal name="ROW_2">
@@
 <wire x1="10.16" y1="73.66" x2="10.16" y2="31.22220625" width="0.2032" layer="1"/>
 <wire x1="10.16" y1="73.66" x2="12.7" y2="76.2" width="0.2032" layer="1"/>
-<wire x1="12.7" y1="76.2" x2="45.72" y2="76.2" width="0.2032" layer="1"/>
-<wire x1="45.72" y1="76.2" x2="48.26" y2="73.66" width="0.2032" layer="1"/>
-<wire x1="48.26" y1="73.66" x2="48.26" y2="67.31" width="0.2032" layer="1"/>
 <wire x1="66.04" y1="24.13" x2="67.31" y2="22.86" width="0.2032" layer="1"/>
 <wire x1="67.31" y1="22.86" x2="78.74" y2="22.86" width="0.2032" layer="1"/>
@@
 <wire x1="10.16" y1="31.22220625" x2="6.84779375" y2="27.91" width="0.2032" layer="1"/>
 <wire x1="6.84779375" y1="27.91" x2="5" y2="27.91" width="0.2032" layer="1"/>
+<wire x1="12.7" y1="76.2" x2="39.37" y2="76.2" width="0.2032" layer="1"/>
+<wire x1="39.37" y1="76.2" x2="48.26" y2="67.31" width="0.2032" layer="1"/>
 </signal>
 <signal name="ROW_3">
@@
 <wire x1="11.43" y1="72.39" x2="11.43" y2="29.21" width="0.2032" layer="1"/>
 <wire x1="11.43" y1="72.39" x2="13.97" y2="74.93" width="0.2032" layer="1"/>
-<wire x1="43.18" y1="74.93" x2="45.72" y2="72.39" width="0.2032" layer="1"/>
-<wire x1="45.72" y1="72.39" x2="45.72" y2="67.31" width="0.2032" layer="1"/>
-<wire x1="13.97" y1="74.93" x2="43.18" y2="74.93" width="0.2032" layer="1"/>
 <wire x1="64.77" y1="22.86" x2="64.77" y2="59.69" width="0.2032" layer="1"/>
 <wire x1="64.77" y1="22.86" x2="67.31" y2="20.32" width="0.2032" layer="1"/>
@@
 <wire x1="6.65" y1="26.66" x2="6.66" y2="26.67" width="0.2032" layer="1"/>
 <wire x1="6.66" y1="26.67" x2="8.89" y2="26.67" width="0.2032" layer="1"/>
+<wire x1="13.97" y1="74.93" x2="38.1" y2="74.93" width="0.2032" layer="1"/>
+<wire x1="38.1" y1="74.93" x2="45.72" y2="67.31" width="0.2032" layer="1"/>
 </signal>
 <signal name="ROW_4">
@@
 <wire x1="12.7" y1="27.94" x2="10.16" y2="25.4" width="0.2032" layer="1"/>
 <wire x1="12.7" y1="71.12" x2="15.24" y2="73.66" width="0.2032" layer="1"/>
-<wire x1="40.64" y1="73.66" x2="43.18" y2="71.12" width="0.2032" layer="1"/>
-<wire x1="43.18" y1="71.12" x2="43.18" y2="67.31" width="0.2032" layer="1"/>
 <wire x1="12.7" y1="27.94" x2="12.7" y2="71.12" width="0.2032" layer="1"/>
-<wire x1="15.24" y1="73.66" x2="40.64" y2="73.66" width="0.2032" layer="1"/>
 <wire x1="43.18" y1="67.31" x2="39.37" y2="63.5" width="0.2032" layer="1"/>
 <wire x1="39.37" y1="63.5" x2="39.37" y2="57.15" width="0.2032" layer="1"/>
@@
 <wire x1="10.16" y1="25.4" x2="10.15" y2="25.41" width="0.2032" layer="1"/>
 <wire x1="10.15" y1="25.41" x2="5" y2="25.41" width="0.2032" layer="1"/>
+<wire x1="15.24" y1="73.66" x2="36.83" y2="73.66" width="0.2032" layer="1"/>
+<wire x1="36.83" y1="73.66" x2="43.18" y2="67.31" width="0.2032" layer="1"/>
 </signal>
 <signal name="ROW_5">
@@
 <wire x1="15.24" y1="25.4" x2="15.24" y2="68.58" width="0.2032" layer="1"/>
 <wire x1="15.24" y1="68.58" x2="17.78" y2="71.12" width="0.2032" layer="1"/>
-<wire x1="17.78" y1="71.12" x2="36.83" y2="71.12" width="0.2032" layer="1"/>
-<wire x1="36.83" y1="71.12" x2="38.1" y2="69.85" width="0.2032" layer="1"/>
-<wire x1="38.1" y1="69.85" x2="38.1" y2="67.31" width="0.2032" layer="1"/>
-<wire x1="38.1" y1="67.31" x2="38.1" y2="55.88" width="0.2032" layer="1"/>
-<wire x1="38.1" y1="55.88" x2="43.18" y2="50.8" width="0.2032" layer="1"/>
+<wire x1="43.18" y1="50.8" x2="38.1" y2="55.88" width="0.2032" layer="1"/>
 <wire x1="43.18" y1="50.8" x2="58.42" y2="50.8" width="0.2032" layer="1"/>
 <wire x1="58.42" y1="50.8" x2="62.23" y2="46.99" width="0.2032" layer="1"/>
@@
 <wire x1="11.48" y1="21.64" x2="6.67" y2="21.64" width="0.2032" layer="1"/>
 <wire x1="6.67" y1="21.64" x2="6.65" y2="21.66" width="0.2032" layer="1"/>
+<wire x1="17.78" y1="71.12" x2="34.29" y2="71.12" width="0.2032" layer="1"/>
+<wire x1="34.29" y1="71.12" x2="38.1" y2="67.31" width="0.2032" layer="1"/>
+<wire x1="38.1" y1="55.88" x2="38.1" y2="67.31" width="0.2032" layer="1"/>
 </signal>
 <signal name="ROW_6">
@@
 <wire x1="16.51" y1="24.13" x2="16.51" y2="67.31" width="0.2032" layer="1"/>
 <wire x1="16.51" y1="67.31" x2="19.05" y2="69.85" width="0.2032" layer="1"/>
-<wire x1="34.29" y1="69.85" x2="35.56" y2="68.58" width="0.2032" layer="1"/>
-<wire x1="35.56" y1="68.58" x2="35.56" y2="67.31" width="0.2032" layer="1"/>
-<wire x1="19.05" y1="69.85" x2="34.29" y2="69.85" width="0.2032" layer="1"/>
 <contactref element="U$4" pad="P$11"/>
 <wire x1="8.82" y1="20.39" x2="5.02" y2="20.39" width="0.2032" layer="1"/>
@@
 <wire x1="17.73" y1="11.48" x2="17.73" y2="6.67" width="0.2032" layer="1"/>
 <wire x1="17.73" y1="6.67" x2="17.71" y2="6.65" width="0.2032" layer="1"/>
+<wire x1="19.05" y1="69.85" x2="33.02" y2="69.85" width="0.2032" layer="1"/>
+<wire x1="33.02" y1="69.85" x2="35.56" y2="67.31" width="0.2032" layer="1"/>
 </signal>
 <signal name="COL_I">
@@
 <wire x1="2.54" y1="10.16" x2="3.81" y2="8.89" width="0.2032" layer="1"/>
 <contactref element="U$1" pad="6"/>
-<wire x1="10.16" y1="78.74" x2="50.8" y2="78.74" width="0.2032" layer="1"/>
-<wire x1="50.8" y1="78.74" x2="53.34" y2="76.2" width="0.2032" layer="1"/>
-<wire x1="53.34" y1="76.2" x2="53.34" y2="67.31" width="0.2032" layer="1"/>
 <contactref element="U$4" pad="P$2"/>
 <wire x1="3.7" y1="31.64" x2="6.63" y2="31.64" width="0.2032" layer="1"/>
@@
 <wire x1="7.62" y1="76.2" x2="10.16" y2="78.74" width="0.2032" layer="1"/>
 <wire x1="7.62" y1="32.63" x2="7.62" y2="76.2" width="0.2032" layer="1"/>
+<wire x1="10.16" y1="78.74" x2="41.91" y2="78.74" width="0.2032" layer="1"/>
+<wire x1="41.91" y1="78.74" x2="53.34" y2="67.31" width="0.2032" layer="1"/>
 </signal>
 <signal name="COL_K">
 <contactref element="U$1" pad="5"/>
-<wire x1="55.88" y1="67.31" x2="55.88" y2="77.47" width="0.2032" layer="1"/>
-<wire x1="8.89" y1="80.01" x2="53.34" y2="80.01" width="0.2032" layer="1"/>
-<wire x1="55.88" y1="77.47" x2="53.34" y2="80.01" width="0.2032" layer="1"/>
 <contactref element="U$4" pad="P$1"/>
 <wire x1="5" y1="32.91" x2="6.35" y2="34.26" width="0.2032" layer="1"/>
-<wire x1="6.35" y1="34.26" x2="6.35" y2="34.29" width="0.2032" layer="1"/>
-<wire x1="6.35" y1="34.29" x2="6.35" y2="77.47" width="0.2032" layer="1"/>
+<wire x1="6.35" y1="34.26" x2="6.35" y2="77.47" width="0.2032" layer="1"/>
 <wire x1="6.35" y1="77.47" x2="8.89" y2="80.01" width="0.2032" layer="1"/>
+<wire x1="8.89" y1="80.01" x2="43.18" y2="80.01" width="0.2032" layer="1"/>
+<wire x1="43.18" y1="80.01" x2="55.88" y2="67.31" width="0.2032" layer="1"/>
 </signal>
 <signal name="COL_L">
@@
 <wire x1="13.97" y1="26.67" x2="13.97" y2="69.85" width="0.2032" layer="1"/>
 <wire x1="13.97" y1="69.85" x2="16.51" y2="72.39" width="0.2032" layer="1"/>
-<wire x1="16.51" y1="72.39" x2="38.1" y2="72.39" width="0.2032" layer="1"/>
-<wire x1="38.1" y1="72.39" x2="40.64" y2="69.85" width="0.2032" layer="1"/>
-<wire x1="40.64" y1="69.85" x2="40.64" y2="67.31" width="0.2032" layer="1"/>
 <contactref element="U$4" pad="P$8"/>
 <wire x1="11.44" y1="24.14" x2="6.67" y2="24.14" width="0.2032" layer="1"/>
 <wire x1="6.67" y1="24.14" x2="6.65" y2="24.16" width="0.2032" layer="1"/>
+<wire x1="16.51" y1="72.39" x2="35.56" y2="72.39" width="0.2032" layer="1"/>
+<wire x1="35.56" y1="72.39" x2="40.64" y2="67.31" width="0.2032" layer="1"/>
 </signal>
 <signal name="VBAT">
 <contactref element="U$1" pad="28"/>
 </signal>
-<signal name="3V">
+<signal name="3V1">
 <contactref element="U$1" pad="2"/>
 </signal>

Commit message: i
Routing:
- net COL_H: track 94.8 -> 93.2 mm
Changed lines of the file:
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@@
 <signal name="COL_G">
 <wire x1="7.62" y1="1.27" x2="5.08" y2="3.81" width="0.2032" layer="16"/>
-<wire x1="5.08" y1="3.81" x2="5" y2="3.89" width="0.2032" layer="16"/>
 <wire x1="7.62" y1="1.27" x2="16.51" y2="1.27" width="0.2032" layer="16"/>
 <wire x1="16.51" y1="1.27" x2="18.98" y2="3.74" width="0.2032" layer="16"/>
@@
 <wire x1="20.32" y1="30.48" x2="7.73" y2="17.89" width="0.2032" layer="16"/>
 <wire x1="20.32" y1="30.48" x2="20.32" y2="54.61" width="0.2032" layer="16"/>
-<wire x1="20.32" y1="54.61" x2="33.02" y2="67.31" width="0.2032" layer="16"/>
+<wire x1="33.02" y1="67.31" x2="20.32" y2="54.61" width="0.2032" layer="16"/>
 <contactref element="U$4" pad="P$13"/>
 <wire x1="7.73" y1="17.89" x2="5.08" y2="17.89" width="0.2032" layer="16"/>
@@
 </signal>
 <signal name="COL_H">
-<wire x1="8.82" y1="20.39" x2="17.73" y2="11.48" width="0.2032" layer="1"/>
 <contactref element="U$1" pad="13"/>
-<wire x1="8.82" y1="20.39" x2="12.77" y2="20.39" width="0.2032" layer="1"/>
+<wire x1="5.02" y1="20.39" x2="12.77" y2="20.39" width="0.2032" layer="1"/>
 <wire x1="12.77" y1="20.39" x2="16.51" y2="24.13" width="0.2032" layer="1"/>
 <wire x1="16.51" y1="24.13" x2="16.51" y2="67.31" width="0.2032" layer="1"/>
 <wire x1="16.51" y1="67.31" x2="19.05" y2="69.85" width="0.2032" layer="1"/>
 <contactref element="U$4" pad="P$11"/>
-<wire x1="8.82" y1="20.39" x2="5.02" y2="20.39" width="0.2032" layer="1"/>
 <wire x1="5.02" y1="20.39" x2="5" y2="20.41" width="0.2032" layer="1"/>
 <contactref element="U$7" pad="P$10"/>
-<wire x1="17.73" y1="11.48" x2="17.73" y2="6.67" width="0.2032" layer="1"/>
-<wire x1="17.73" y1="6.67" x2="17.71" y2="6.65" width="0.2032" layer="1"/>
 <wire x1="19.05" y1="69.85" x2="33.02" y2="69.85" width="0.2032" layer="1"/>
 <wire x1="33.02" y1="69.85" x2="35.56" y2="67.31" width="0.2032" layer="1"/>
+<wire x1="12.77" y1="20.39" x2="17.71" y2="15.45" width="0.2032" layer="1"/>
+<wire x1="17.71" y1="15.45" x2="17.71" y2="6.65" width="0.2032" layer="1"/>
 </signal>
 <signal name="COL_I">

Commit message: i
Routing:
- net COL_G: track 94.0 -> 102.9 mm
- net COL_I: track 76.3 -> 85.2 mm
- net ROW_6: track 113.4 -> 107.5 mm
- net ROW_4: track 177.2 -> 176.2 mm
- net ROW_7: track 112.1 -> 111.6 mm

Commit message: i
Routing:
- net COL_F: track 80.2 -> 84.9 mm
- net COL_A: track 63.8 -> 68.2 mm
- net COL_C: track 102.2 -> 106.7 mm
- net COL_B: track 62.4 -> 66.8 mm
- net COL_E: track 101.8 -> 106.3 mm
- net COL_D: track 76.6 -> 81.0 mm
- net ROW_4: track 176.2 -> 177.2 mm
Changed lines of the file:
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@@
 <wire x1="15.24" y1="73.66" x2="36.83" y2="73.66" width="0.2032" layer="1"/>
 <wire x1="36.83" y1="73.66" x2="43.18" y2="67.31" width="0.2032" layer="1"/>
-<wire x1="43.18" y1="67.31" x2="43.18" y2="66.04" width="0.2032" layer="1"/>
-<wire x1="40.64" y1="63.5" x2="40.64" y2="54.61" width="0.2032" layer="1"/>
-<wire x1="40.64" y1="54.61" x2="44.45" y2="50.8" width="0.2032" layer="1"/>
-<wire x1="43.18" y1="66.04" x2="40.64" y2="63.5" width="0.2032" layer="1"/>
 <wire x1="73.66" y1="50.8" x2="76.2" y2="48.26" width="0.2032" layer="1"/>
 <wire x1="76.2" y1="48.26" x2="76.2" y2="22.86" width="0.2032" layer="1"/>
@@
 <wire x1="81.28" y1="19.05" x2="87.24" y2="19.05" width="0.2032" layer="16"/>
 <wire x1="87.24" y1="19.05" x2="87.33" y2="19.14" width="0.2032" layer="16"/>
+<wire x1="43.18" y1="67.31" x2="39.37" y2="63.5" width="0.2032" layer="1"/>
+<wire x1="39.37" y1="63.5" x2="39.37" y2="55.88" width="0.2032" layer="1"/>
+<wire x1="39.37" y1="55.88" x2="44.45" y2="50.8" width="0.2032" layer="1"/>
 </signal>
 <signal name="ROW_5">
@@
 <wire x1="17.78" y1="71.12" x2="34.29" y2="71.12" width="0.2032" layer="1"/>
 <wire x1="34.29" y1="71.12" x2="38.1" y2="67.31" width="0.2032" layer="1"/>
-<wire x1="38.1" y1="67.31" x2="39.37" y2="66.04" width="0.2032" layer="1"/>
-<wire x1="39.37" y1="53.34" x2="43.18" y2="49.53" width="0.2032" layer="1"/>
-<wire x1="39.37" y1="66.04" x2="39.37" y2="53.34" width="0.2032" layer="1"/>
 <wire x1="72.39" y1="49.53" x2="74.93" y2="46.99" width="0.2032" layer="1"/>
 <wire x1="74.93" y1="46.99" x2="74.93" y2="21.59" width="0.2032" layer="1"/>
@@
 <wire x1="81.28" y1="17.78" x2="88.87" y2="17.78" width="0.2032" layer="16"/>
 <wire x1="88.87" y1="17.78" x2="88.98" y2="17.89" width="0.2032" layer="16"/>
+<wire x1="38.1" y1="67.31" x2="38.1" y2="54.61" width="0.2032" layer="1"/>
+<wire x1="38.1" y1="54.61" x2="43.18" y2="49.53" width="0.2032" layer="1"/>
 </signal>
 <signal name="ROW_6">
@@
 <contactref element="U$5" pad="P$6"/>
 <contactref element="U$1" pad="19"/>
-<wire x1="33.02" y1="46.99" x2="55.87" y2="24.14" width="0.2032" layer="16"/>
-<wire x1="55.87" y1="24.14" x2="87.33" y2="24.14" width="0.2032" layer="16"/>
+<wire x1="33.02" y1="46.99" x2="41.91" y2="38.1" width="0.2032" layer="16"/>
+<wire x1="76.2" y1="38.1" x2="78.74" y2="35.56" width="0.2032" layer="16"/>
+<wire x1="78.74" y1="27.94" x2="82.55" y2="24.13" width="0.2032" layer="16"/>
+<wire x1="82.55" y1="24.13" x2="82.56" y2="24.14" width="0.2032" layer="16"/>
+<wire x1="82.56" y1="24.14" x2="87.33" y2="24.14" width="0.2032" layer="16"/>
+<wire x1="41.91" y1="38.1" x2="76.2" y2="38.1" width="0.2032" layer="16"/>
+<wire x1="78.74" y1="35.56" x2="78.74" y2="27.94" width="0.2032" layer="16"/>
 </signal>
 <signal name="COL_B">
 <contactref element="U$5" pad="P$7"/>
 <contactref element="U$1" pad="20"/>
-<wire x1="35.56" y1="46.99" x2="57.16" y2="25.39" width="0.2032" layer="16"/>
-<wire x1="57.16" y1="25.39" x2="88.98" y2="25.39" width="0.2032" layer="16"/>
+<wire x1="35.56" y1="46.99" x2="43.18" y2="39.37" width="0.2032" layer="16"/>
+<wire x1="77.47" y1="39.37" x2="80.01" y2="36.83" width="0.2032" layer="16"/>
+<wire x1="80.01" y1="36.83" x2="80.01" y2="29.21" width="0.2032" layer="16"/>
+<wire x1="43.18" y1="39.37" x2="77.47" y2="39.37" width="0.2032" layer="16"/>
+<wire x1="83.83" y1="25.39" x2="88.98" y2="25.39" width="0.2032" layer="16"/>
+<wire x1="80.01" y1="29.21" x2="83.83" y2="25.39" width="0.2032" layer="16"/>
 </signal>
 <signal name="COL_C">
@@
 <wire x1="74.93" y1="2.54" x2="73.75" y2="3.72" width="0.2032" layer="16"/>
 <contactref element="U$1" pad="22"/>
-<wire x1="40.64" y1="46.99" x2="60.99" y2="26.64" width="0.2032" layer="16"/>
-<wire x1="60.99" y1="26.64" x2="87.33" y2="26.64" width="0.2032" layer="16"/>
+<wire x1="40.64" y1="46.99" x2="46.99" y2="40.64" width="0.2032" layer="16"/>
+<wire x1="78.74" y1="40.64" x2="81.28" y2="38.1" width="0.2032" layer="16"/>
+<wire x1="81.28" y1="30.48" x2="85.12" y2="26.64" width="0.2032" layer="16"/>
+<wire x1="85.12" y1="26.64" x2="87.33" y2="26.64" width="0.2032" layer="16"/>
+<wire x1="46.99" y1="40.64" x2="78.74" y2="40.64" width="0.2032" layer="16"/>
+<wire x1="81.28" y1="38.1" x2="81.28" y2="30.48" width="0.2032" layer="16"/>
 </signal>
 <signal name="COL_D">
@@
 <wire x1="85.09" y1="10.49" x2="85.09" y2="26.9" width="0.2032" layer="1"/>
 <contactref element="U$1" pad="23"/>
-<wire x1="43.18" y1="46.99" x2="61.03" y2="29.14" width="0.2032" layer="16"/>
-<wire x1="61.03" y1="29.14" x2="87.33" y2="29.14" width="0.2032" layer="16"/>
+<wire x1="43.18" y1="46.99" x2="48.26" y2="41.91" width="0.2032" layer="16"/>
+<wire x1="80.01" y1="41.91" x2="82.55" y2="39.37" width="0.2032" layer="16"/>
+<wire x1="82.55" y1="39.37" x2="82.55" y2="31.75" width="0.2032" layer="16"/>
+<wire x1="82.55" y1="31.75" x2="85.16" y2="29.14" width="0.2032" layer="16"/>
+<wire x1="85.16" y1="29.14" x2="87.33" y2="29.14" width="0.2032" layer="16"/>
+<wire x1="48.26" y1="41.91" x2="80.01" y2="41.91" width="0.2032" layer="16"/>
 </signal>
 <signal name="COL_E">
@@
 <wire x1="72.5" y1="3.7" x2="74.93" y2="1.27" width="0.2032" layer="16"/>
 <contactref element="U$1" pad="24"/>
-<wire x1="45.72" y1="46.99" x2="62.32" y2="30.39" width="0.2032" layer="16"/>
-<wire x1="62.32" y1="30.39" x2="88.98" y2="30.39" width="0.2032" layer="16"/>
+<wire x1="45.72" y1="46.99" x2="49.53" y2="43.18" width="0.2032" layer="16"/>
+<wire x1="81.28" y1="43.18" x2="83.82" y2="40.64" width="0.2032" layer="16"/>
+<wire x1="83.82" y1="40.64" x2="83.82" y2="33.02" width="0.2032" layer="16"/>
+<wire x1="83.82" y1="33.02" x2="86.45" y2="30.39" width="0.2032" layer="16"/>
+<wire x1="86.45" y1="30.39" x2="88.98" y2="30.39" width="0.2032" layer="16"/>
+<wire x1="49.53" y1="43.18" x2="81.28" y2="43.18" width="0.2032" layer="16"/>
 </signal>
 <signal name="COL_F">
@@
 <wire x1="87.33" y1="31.45" x2="87.33" y2="31.64" width="0.2032" layer="1"/>
 <contactref element="U$1" pad="25"/>
-<wire x1="48.26" y1="46.99" x2="63.61" y2="31.64" width="0.2032" layer="16"/>
-<wire x1="63.61" y1="31.64" x2="87.33" y2="31.64" width="0.2032" layer="16"/>
+<wire x1="48.26" y1="46.99" x2="50.8" y2="44.45" width="0.2032" layer="16"/>
+<wire x1="50.8" y1="44.45" x2="82.55" y2="44.45" width="0.2032" layer="16"/>
+<wire x1="82.55" y1="44.45" x2="85.09" y2="41.91" width="0.2032" layer="16"/>
+<wire x1="85.09" y1="41.91" x2="85.09" y2="33.88" width="0.2032" layer="16"/>
+<wire x1="85.09" y1="33.88" x2="87.33" y2="31.64" width="0.2032" layer="16"/>
 </signal>
 <signal name="COL_G">
