File: hardware/controller.brd (EAGLE design)
At the start: 94.1 x 81.3 mm, 5 parts

Commit message: i
Parts:
- moved U$4 45.1 mm to (5.08, 70.5)
- moved U$5 45.1 mm to (88.9, 70.5)
- moved U$6 45.1 mm to (80.0, 50.2)
- moved U$7 45.1 mm to (14.0, 50.2)
- moved U$1 33.0 mm to (47.0, 24.1), turned to 90 degrees
Connections:
- new net GND: U$1.4
Routing:
- net ROW_4: track 177.2 -> 0.00 mm, vias 1 -> 0
- net ROW_5: track 172.6 -> 0.00 mm, vias 1 -> 0
- net ROW_2: track 172.5 -> 0.00 mm, vias 1 -> 0
- net ROW_3: track 171.8 -> 0.00 mm, vias 1 -> 0
- net COL_K: track 101.0 -> 0.00 mm
- net COL_J: track 135.5 -> 39.0 mm
- net ROW_1: track 93.9 -> 0.00 mm
- net COL_L: track 81.4 -> 0.00 mm
- net COL_G: track 102.9 -> 28.7 mm
- net COL_H: track 93.2 -> 20.5 mm
- net COL_A: track 68.2 -> 0.00 mm
- net COL_B: track 66.8 -> 0.00 mm
- net COL_I: track 85.2 -> 18.7 mm
- net COL_C: track 106.7 -> 47.1 mm
- net COL_E: track 106.3 -> 49.9 mm
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Other:
- board size 94.1 x 81.3 mm -> 94 x 126.4 mm

Commit message: i
Connections:
- net COL_A: now also U$1.8; no longer U$1.19
- net COL_B: now also U$1.9; no longer U$1.20
- net COL_C: now also U$1.14; no longer U$1.22
- net COL_D: now also U$1.10; no longer U$1.23
- net COL_E: now also U$1.15; no longer U$1.24
- net COL_F: now also U$1.13; no longer U$1.25
- net COL_G: now also U$1.17; no longer U$1.14
- net COL_H: now also U$1.18; no longer U$1.13
- net COL_I: now also U$1.19; no longer U$1.15
- net COL_K: now also U$1.7; no longer U$1.5
- net COL_L: now also U$1.22; no longer U$1.11
- net ROW_1: now also U$1.5; no longer U$1.7
- net ROW_2: now also U$1.25; no longer U$1.8
- net ROW_3: now also U$1.24; no longer U$1.9
- net ROW_4: now also U$1.23; no longer U$1.10
- net ROW_5: now also U$1.20; no longer U$1.12
- net ROW_6: now also U$1.11; no longer U$1.18
- net ROW_7: now also U$1.12; no longer U$1.17
Routing:
- net ROW_2: track 0.00 -> 172.2 mm
- net ROW_3: track 0.00 -> 160.9 mm
- net ROW_4: track 0.00 -> 155.6 mm
- net ROW_5: track 0.00 -> 130.2 mm
- net COL_K: track 0.00 -> 89.9 mm
- net ROW_1: track 0.00 -> 89.7 mm
- net COL_J: track 39.0 -> 128.4 mm
- net COL_A: track 0.00 -> 83.8 mm
- net COL_B: track 0.00 -> 81.3 mm
- net COL_L: track 0.00 -> 63.4 mm
- net COL_D: track 25.0 -> 79.8 mm
- net ROW_6: track 70.0 -> 117.1 mm
- net ROW_7: track 67.0 -> 106.1 mm
- net COL_F: track 34.7 -> 72.1 mm
- net COL_I: track 18.7 -> 55.4 mm
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Other:
- board size 94 x 126.4 mm -> 94 x 127 mm

Commit message: i
Other:
- board size 94 x 127 mm -> 94 x 111.1 mm
- board text added: "02/14/2019"
- board text added: "FeatherCtrl v2"
- board text removed: "FeatherCtrl"
Changed lines of the file:
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@@
 <wire x1="59.055" y1="44.45" x2="91.811978125" y2="44.45" width="0" layer="20"/>
 <wire x1="91.811978125" y1="44.45" x2="93.98" y2="46.618021875" width="0" layer="20" curve="90"/>
-<wire x1="93.98" y1="46.618021875" x2="93.98" y2="124.19664375" width="0" layer="20"/>
-<wire x1="93.98" y1="124.19664375" x2="91.81164375" y2="126.365484375" width="0" layer="20" curve="89.987204"/>
-<wire x1="91.81164375" y1="126.365484375" x2="2.20340625" y2="126.38550625" width="0" layer="20"/>
-<wire x1="2.20340625" y1="126.38550625" x2="0" y2="124.18259375" width="0" layer="20" curve="89.837974"/>
-<wire x1="0" y1="124.18259375" x2="0" y2="46.618021875" width="0" layer="20"/>
+<wire x1="93.98" y1="46.618021875" x2="93.98" y2="108.32164375" width="0" layer="20"/>
+<wire x1="93.98" y1="108.32164375" x2="91.81164375" y2="110.490484375" width="0" layer="20" curve="89.987204"/>
+<wire x1="91.81164375" y1="110.490484375" x2="2.20340625" y2="110.51050625" width="0" layer="20"/>
+<wire x1="2.20340625" y1="110.51050625" x2="0" y2="108.30759375" width="0" layer="20" curve="89.837974"/>
+<wire x1="0" y1="108.30759375" x2="0" y2="46.618021875" width="0" layer="20"/>
 <wire x1="0" y1="46.618021875" x2="2.168021875" y2="44.45" width="0" layer="20" curve="90"/>
 <wire x1="2.168021875" y1="44.45" x2="34.925" y2="44.45" width="0" layer="20"/>
 <hole x="47.03" y="102.775" drill="6.4"/>
 <hole x="47.03" y="71.275" drill="4.1"/>
-<text x="80.01" y="86.995" size="2.54" layer="21" rot="R180">FeatherCtrl</text>
+<text x="80.01" y="86.995" size="2.54" layer="21" rot="R180">FeatherCtrl v2</text>
 <text x="80.01" y="80.645" size="1.4224" layer="21" rot="R180">github.com/matthewvilim/featherctrl</text>
 <text x="80.01" y="83.185" size="1.4224" layer="21" rot="R180">Matthew Vilim</text>
-<wire x1="34.925" y1="44.45" x2="34.925" y2="1.533021875" width="0" layer="20"/>
-<wire x1="34.925" y1="1.533021875" x2="37.093021875" y2="-0.635" width="0" layer="20" curve="90"/>
-<wire x1="37.093021875" y1="-0.635" x2="56.886978125" y2="-0.635" width="0" layer="20"/>
-<wire x1="56.886978125" y1="-0.635" x2="59.055" y2="1.533021875" width="0" layer="20" curve="90"/>
-<wire x1="59.055" y1="1.533021875" x2="59.055" y2="44.45" width="0" layer="20"/>
+<wire x1="34.925" y1="44.45" x2="34.925" y2="2.54" width="0" layer="20"/>
+<wire x1="34.925" y1="2.54" x2="38.1" y2="-0.635" width="0" layer="20" curve="90"/>
+<wire x1="38.1" y1="-0.635" x2="55.88" y2="-0.635" width="0" layer="20"/>
+<wire x1="55.88" y1="-0.635" x2="59.055" y2="2.54" width="0" layer="20" curve="90"/>
+<wire x1="59.055" y1="2.54" x2="59.055" y2="44.45" width="0" layer="20"/>
+<text x="80.01" y="78.105" size="1.4224" layer="21" rot="R180">02/14/2019</text>
 </plain>
 <attributes>
@@
 <wire x1="36.83" y1="24.13" x2="41.91" y2="29.21" width="0.254" layer="16"/>
 <wire x1="41.91" y1="50.165" x2="34.925" y2="57.15" width="0.254" layer="16"/>
-<wire x1="16.51" y1="57.15" x2="11.43" y2="62.23" width="0.254" layer="16"/>
-<wire x1="5.2404" y1="72.7546" x2="5" y2="72.995" width="0.254" layer="16"/>
-<wire x1="7.06819375" y1="72.7546" x2="5.2404" y2="72.7546" width="0.254" layer="16"/>
-<wire x1="11.43" y1="68.39279375" x2="7.06819375" y2="72.7546" width="0.254" layer="16"/>
-<wire x1="11.43" y1="62.23" x2="11.43" y2="68.39279375" width="0.254" layer="16"/>
+<wire x1="11.43" y1="62.23" x2="16.51" y2="57.15" width="0.254" layer="16"/>
 <wire x1="41.91" y1="29.21" x2="41.91" y2="50.165" width="0.254" layer="16"/>
 <wire x1="34.925" y1="57.15" x2="16.51" y2="57.15" width="0.254" layer="16"/>
-<wire x1="88.98" y1="67.975" x2="88.98" y2="66.9387125" width="0.254" layer="1"/>
-<wire x1="88.98" y1="66.9387125" x2="91.2622" y2="64.6565125" width="0.254" layer="1"/>
 <wire x1="43.18" y1="45.72" x2="40.64" y2="43.18" width="0.254" layer="1"/>
 <wire x1="40.64" y1="27.94" x2="36.83" y2="24.13" width="0.254" layer="1"/>
-<wire x1="91.2622" y1="64.6565125" x2="91.2622" y2="48.0822" width="0.254" layer="1"/>
 <wire x1="91.2622" y1="48.0822" x2="88.9" y2="45.72" width="0.254" layer="1"/>
 <wire x1="88.9" y1="45.72" x2="43.18" y2="45.72" width="0.254" layer="1"/>
 <wire x1="40.64" y1="43.18" x2="40.64" y2="27.94" width="0.254" layer="1"/>
+<wire x1="88.98" y1="67.975" x2="91.2622" y2="65.6928" width="0.254" layer="1"/>
+<wire x1="91.2622" y1="65.6928" x2="91.2622" y2="48.0822" width="0.254" layer="1"/>
+<wire x1="6.8637125" y1="72.995" x2="11.43" y2="68.4287125" width="0.254" layer="16"/>
+<wire x1="5" y1="72.995" x2="6.8637125" y2="72.995" width="0.254" layer="16"/>
+<wire x1="11.43" y1="68.4287125" x2="11.43" y2="62.23" width="0.254" layer="16"/>
 </signal>
 <signal name="ROW_3">
@@
 <wire x1="40.64" y1="48.895" x2="33.655" y2="55.88" width="0.254" layer="16"/>
 <wire x1="33.655" y1="55.88" x2="15.24" y2="55.88" width="0.254" layer="16"/>
-<wire x1="15.24" y1="55.88" x2="10.16" y2="60.96" width="0.254" layer="16"/>
-<wire x1="10.16" y1="67.16279375" x2="6.82779375" y2="70.495" width="0.254" layer="16"/>
-<wire x1="6.82779375" y1="70.495" x2="5" y2="70.495" width="0.254" layer="16"/>
-<wire x1="10.16" y1="60.96" x2="10.16" y2="67.16279375" width="0.254" layer="16"/>
+<wire x1="10.16" y1="60.96" x2="15.24" y2="55.88" width="0.254" layer="16"/>
 <wire x1="87.33" y1="64.225" x2="87.545" y2="64.01" width="0.254" layer="1"/>
 <wire x1="87.545" y1="64.01" x2="89.4087125" y2="64.01" width="0.254" layer="1"/>
@@
 <wire x1="39.37" y1="31.75" x2="36.83" y2="29.21" width="0.254" layer="1"/>
 <wire x1="87.63" y1="46.99" x2="41.91" y2="46.99" width="0.254" layer="1"/>
+<wire x1="5" y1="70.495" x2="6.975" y2="70.495" width="0.254" layer="16"/>
+<wire x1="6.975" y1="70.495" x2="10.16" y2="67.31" width="0.254" layer="16"/>
+<wire x1="10.16" y1="67.31" x2="10.16" y2="60.96" width="0.254" layer="16"/>
 </signal>
 <signal name="ROW_5">
@@
 <contactref element="U$6" pad="P$4"/>
 <contactref element="U$7" pad="P$7"/>
-<wire x1="76.2" y1="51.685" x2="76.25" y2="51.735" width="0.254" layer="1"/>
 <contactref element="U$1" pad="12"/>
 <wire x1="57.15" y1="34.29" x2="53.975" y2="37.465" width="0.254" layer="16"/>
@@
 <wire x1="74.645" y1="53.34" x2="76.25" y2="51.735" width="0.254" layer="16"/>
 <wire x1="57.785" y1="53.34" x2="74.645" y2="53.34" width="0.254" layer="16"/>
-<wire x1="75.4287125" y1="49.05" x2="76.035" y2="49.6562875" width="0.254" layer="1"/>
 <wire x1="13.96" y1="50.085" x2="14.9962875" y2="50.085" width="0.254" layer="1"/>
-<wire x1="76.035" y1="51.52" x2="76.25" y2="51.735" width="0.254" layer="1"/>
 <wire x1="14.9962875" y1="50.085" x2="16.0312875" y2="49.05" width="0.254" layer="1"/>
-<wire x1="76.035" y1="49.6562875" x2="76.035" y2="51.52" width="0.254" layer="1"/>
 <wire x1="16.0312875" y1="49.05" x2="75.4287125" y2="49.05" width="0.254" layer="1"/>
+<wire x1="75.4287125" y1="49.05" x2="76.25" y2="49.8712875" width="0.254" layer="1"/>
+<wire x1="76.25" y1="49.8712875" x2="76.25" y2="51.735" width="0.254" layer="1"/>
 </signal>
 <signal name="COL_A">
@@
 <signal name="GND">
 <polygon width="0.254" layer="1" isolate="0.254">
-<vertex x="91.811978125" y="126.365"/>
-<vertex x="2.168021875" y="126.365" curve="90"/>
-<vertex x="0" y="124.196978125"/>
+<vertex x="91.811978125" y="110.49"/>
+<vertex x="2.168021875" y="110.49" curve="90"/>
+<vertex x="0" y="108.321978125"/>
 <vertex x="0" y="46.618021875" curve="90"/>
 <vertex x="2.168021875" y="44.45"/>
 <vertex x="34.925" y="44.45"/>
-<vertex x="34.925" y="1.533021875" curve="90"/>
-<vertex x="37.093021875" y="-0.635"/>
-<vertex x="56.886978125" y="-0.635" curve="90"/>
-<vertex x="59.055" y="1.533021875"/>
+<vertex x="34.925" y="2.54" curve="90"/>
+<vertex x="38.1" y="-0.635"/>
+<vertex x="55.88" y="-0.635" curve="90"/>
+<vertex x="59.055" y="2.54"/>
 <vertex x="59.055" y="44.45"/>
 <vertex x="91.811978125" y="44.45" curve="90"/>
 <vertex x="93.98" y="46.618021875"/>
-<vertex x="93.98" y="124.196978125" curve="90"/>
+<vertex x="93.98" y="108.321978125" curve="90"/>
 </polygon>
 <polygon width="0.254" layer="16" isolate="0.254">
@@
 <vertex x="2.168021875" y="44.45" curve="-90"/>
 <vertex x="0" y="46.618021875"/>
-<vertex x="0" y="124.196978125" curve="-90"/>
-<vertex x="2.168021875" y="126.365"/>
-<vertex x="91.811978125" y="126.365" curve="-90"/>
-<vertex x="93.98" y="124.196978125"/>
+<vertex x="0" y="108.321978125" curve="-90"/>
+<vertex x="2.168021875" y="110.49"/>
+<vertex x="91.811978125" y="110.49" curve="-90"/>
+<vertex x="93.98" y="108.321978125"/>
 <vertex x="93.98" y="46.618021875" curve="-90"/>
 <vertex x="91.811978125" y="44.45"/>
 <vertex x="59.055" y="44.45"/>
-<vertex x="59.055" y="1.533021875" curve="-90"/>
-<vertex x="56.886978125" y="-0.635"/>
-<vertex x="37.093021875" y="-0.635" curve="-90"/>
-<vertex x="34.925" y="1.533021875"/>
+<vertex x="59.055" y="2.54" curve="-90"/>
+<vertex x="55.88" y="-0.635"/>
+<vertex x="38.1" y="-0.635" curve="-90"/>
+<vertex x="34.925" y="2.54"/>
 </polygon>
 <contactref element="U$1" pad="4"/>

Commit message: i
Routing:
- net COL_J: track 128.4 -> 124.3 mm
Changed lines of the file:
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@@
 </signal>
 <signal name="COL_J">
-<wire x1="2.54" y1="75.565" x2="3.7" y2="76.725" width="0.254" layer="1"/>
-<wire x1="2.54" y1="75.565" x2="2.54" y2="55.245" width="0.254" layer="1"/>
-<wire x1="2.54" y1="55.245" x2="3.81" y2="53.975" width="0.254" layer="1"/>
 <contactref element="U$1" pad="6"/>
 <contactref element="U$4" pad="P$2"/>
-<wire x1="3.7" y1="76.725" x2="6.63" y2="76.725" width="0.254" layer="1"/>
-<wire x1="6.65" y1="76.745" x2="6.63" y2="76.725" width="0.254" layer="1"/>
 <contactref element="U$7" pad="P$8"/>
-<wire x1="12.97" y1="53.975" x2="15.21" y2="51.735" width="0.254" layer="1"/>
-<wire x1="3.81" y1="53.975" x2="12.97" y2="53.975" width="0.254" layer="1"/>
 <wire x1="57.15" y1="19.05" x2="43.18" y2="33.02" width="0.254" layer="16"/>
 <wire x1="36.195" y1="58.42" x2="17.78" y2="58.42" width="0.254" layer="16"/>
@@
 <wire x1="43.18" y1="51.435" x2="36.195" y2="58.42" width="0.254" layer="16"/>
 <wire x1="12.7" y1="63.5" x2="12.7" y2="70.695" width="0.254" layer="16"/>
+<wire x1="6.65" y1="76.745" x2="4.355" y2="76.745" width="0.254" layer="1"/>
+<wire x1="4.355" y1="76.745" x2="3.81" y2="76.2" width="0.254" layer="1"/>
+<wire x1="3.81" y1="76.2" x2="3.81" y2="62.23" width="0.254" layer="1"/>
+<wire x1="5.715" y1="60.325" x2="10.16" y2="60.325" width="0.254" layer="1"/>
+<wire x1="10.16" y1="60.325" x2="15.21" y2="55.275" width="0.254" layer="1"/>
+<wire x1="15.21" y1="55.275" x2="15.21" y2="51.735" width="0.254" layer="1"/>
+<wire x1="3.81" y1="62.23" x2="5.715" y2="60.325" width="0.254" layer="1"/>
 </signal>
 <signal name="COL_K">

Commit message: i
Routing:
- net COL_C: track 76.7 -> 75.5 mm
- net COL_E: track 73.8 -> 72.5 mm
Other:
- board size 94 x 111.1 mm -> 94 x 84.5 mm

Commit message: i
Routing:
- net COL_L: track 63.4 -> 64.7 mm
- net ROW_2: track 172.6 -> 173.9 mm
- net ROW_3: track 161.3 -> 162.4 mm
- net ROW_4: track 156.1 -> 157.2 mm
- net ROW_1: track 89.7 -> 90.8 mm
- net ROW_5: track 130.2 -> 131.1 mm
- net COL_J: track 124.3 -> 124.9 mm
- net COL_K: track 89.9 -> 90.4 mm
Other:
- board text added: "FeatherCtrl"
- board text added: "Feb 2019 v2"
- board text removed: "02/14/2019"
- board text removed: "FeatherCtrl v2"
