File: hardware/controller.sch (EAGLE design)
At the start: 5 parts

Commit message: i
Parts:
- U$1: device mike:NRF52FEATHER -> adafruit:NRF52FEATHER
Connections:
- removed net N$19: U$5.P$9
- removed net N$24: U$5.P$4
- removed net N$44: U$4.P$5
- removed net N$50: U$4.P$11
- removed net N$54: U$6.P$13
- removed net N$55: U$6.P$11
- removed net N$56: U$6.P$12
- removed net N$57: U$6.P$10
- removed net N$58: U$6.P$9
- removed net N$60: U$6.P$7
- removed net N$61: U$6.P$6
- removed net N$67: U$7.P$1
- removed net N$68: U$7.P$2
- removed net N$75: U$7.P$9
- removed net N$76: U$7.P$10
- removed net N$77: U$7.P$11
- removed net N$78: U$7.P$12
- removed net N$79: U$7.P$13
- net COL_G: now also U$4.P$13, U$7.P$11; no longer U$4.P$1, U$7.P$3
- net COL_H: now also U$4.P$11, U$7.P$10; no longer U$4.P$3, U$7.P$4
- net COL_I: now also U$4.P$12, U$7.P$9; no longer U$4.P$2, U$7.P$5
- net COL_J: now also U$4.P$2, U$7.P$8; no longer U$4.P$12, U$7.P$6
- net COL_K: now also U$4.P$1; no longer U$4.P$13
- net COL_L: now also U$4.P$8; no longer U$4.P$6
- net ROW_1: now also U$4.P$4; no longer U$4.P$10
- net ROW_2: now also U$4.P$5; no longer U$4.P$9
- net ROW_3: now also U$4.P$6; no longer U$4.P$8
- net ROW_5: now also U$4.P$10; no longer U$4.P$4
- net ROW_6: now also U$7.P$6; no longer U$7.P$8
