File: hardware/controller.sch (EAGLE design)
At the start: 5 parts

Commit message: i
Connections:
- removed net 3V: U$1.3V@1
- removed net 3V2: U$1.3V@2
Changed lines of the file:
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@@
-</segment>
-</net>
-<net name="3V" class="0">
-<segment>
-<pinref part="U$1" gate="G$1" pin="3V@1"/>
-<wire x1="81.28" y1="58.42" x2="81.28" y2="68.58" width="0.1524" layer="91"/>
-<label x="81.28" y="60.96" size="1.778" layer="95" rot="R90"/>
-</segment>
-</net>
-<net name="3V2" class="0">
-<segment>
-<pinref part="U$1" gate="G$1" pin="3V@2"/>
-<wire x1="78.74" y1="58.42" x2="78.74" y2="68.58" width="0.1524" layer="91"/>
-<label x="78.74" y="60.96" size="1.778" layer="95" rot="R90"/>
 </segment>
 </net>

Commit message: i
Connections:
- new net GND: U$1.GND
Changed lines of the file:
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@@
 <?xml version="1.0" encoding="utf-8"?>
 <!DOCTYPE eagle SYSTEM "eagle.dtd">
-<eagle version="9.2.2">
+<eagle version="9.3.0">
 <drawing>
 <settings>
@@
 </segment>
 </net>
+<net name="GND" class="0">
+<segment>
+<pinref part="U$1" gate="G$1" pin="GND"/>
+<wire x1="76.2" y1="58.42" x2="76.2" y2="68.58" width="0.1524" layer="91"/>
+<label x="76.2" y="68.58" size="1.778" layer="95" rot="R270"/>
+</segment>
+</net>

Commit message: i
Connections:
- net COL_A: now also U$1.A3; no longer U$1.27
- net COL_B: now also U$1.A4; no longer U$1.30A6
- net COL_C: now also U$1.RX; no longer U$1.11
- net COL_D: now also U$1.A5; no longer U$1.7
- net COL_E: now also U$1.TX; no longer U$1.15
- net COL_F: now also U$1.MISO; no longer U$1.16
- net COL_G: now also U$1.SDA; no longer U$1.RX
- net COL_H: now also U$1.SCL; no longer U$1.MISO
- net COL_I: now also U$1.27; no longer U$1.TX
- net COL_K: now also U$1.A2; no longer U$1.A0
- net COL_L: now also U$1.11; no longer U$1.SCK
- net ROW_1: now also U$1.A0; no longer U$1.A2
- net ROW_2: now also U$1.16; no longer U$1.A3
- net ROW_3: now also U$1.15; no longer U$1.A4
- net ROW_4: now also U$1.7; no longer U$1.A5
- net ROW_5: now also U$1.30A6; no longer U$1.MOSI
- net ROW_6: now also U$1.SCK; no longer U$1.SCL
- net ROW_7: now also U$1.MOSI; no longer U$1.SDA
